File: arduino/kicad/mega2560/tester.kicad_sch (KiCad schematic)
At the start: 37 parts, among them J1 AudioJack2, J1 Conn_01x08, J2 AudioJack2, J2 Conn_01x08, J3 Conn_01x10, J3 XLR3, J4 Conn_01x08, J4 XLR3, J5 Conn_01x08, J6 Conn_01x08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

Commit message: kicad and pricing util
Connections:
- net D15 is gone; now on net GND: D3.2 (A), J1.7 (D15), K3.A2
- net D16: now also K4.A1; no longer K4.A2
- net D63: now also D8.2 (A); no longer D8.1 (K)
- net GND: now also D8.1 (K), K4.A2; no longer D8.2 (A), K4.A1
Other:
- moved on the sheet: D3
Changed lines of the file:
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@@
 	)
 	(junction
-		(at 96.52 161.29)
+		(at 63.5 102.87)
 		(diameter 0)
 		(color 0 0 0 0)
 	)
 	(junction
-		(at 63.5 102.87)
+		(at 96.52 181.61)
 		(diameter 0)
 		(color 0 0 0 0)
@@
 	)
 	(junction
+		(at 205.74 168.91)
+		(diameter 0)
+		(color 0 0 0 0)
+	)
+	(junction
 		(at 285.75 148.59)
 		(diameter 0)
@@
 	)
 	(junction
-		(at 130.81 160.02)
+		(at 90.17 181.61)
+		(diameter 0)
+		(color 0 0 0 0)
+	)
+	(junction
+		(at 83.82 161.29)
 		(diameter 0)
 		(color 0 0 0 0)
 	)
 	(junction
-		(at 226.06 168.91)
+		(at 226.06 154.94)
 		(diameter 0)
 		(color 0 0 0 0)
 	)
 	(junction
-		(at 83.82 161.29)
+		(at 130.81 160.02)
 		(diameter 0)
 		(color 0 0 0 0)
@@
 	)
 	(junction
-		(at 205.74 168.91)
+		(at 285.75 106.68)
 		(diameter 0)
 		(color 0 0 0 0)
 	)
 	(junction
-		(at 285.75 106.68)
+		(at 90.17 161.29)
 		(diameter 0)
 		(color 0 0 0 0)
@@
 	(wire
 		(pts
-			(xy 242.57 176.53) (xy 223.52 176.53)
+			(xy 90.17 175.26) (xy 90.17 181.61)
 		)
 		(stroke
@@
 	(wire
 		(pts
-			(xy 237.49 162.56) (xy 264.16 162.56)
+			(xy 242.57 176.53) (xy 223.52 176.53)
 		)
 		(stroke
@@
 	(wire
 		(pts
-			(xy 129.54 36.83) (xy 162.56 36.83)
+			(xy 237.49 162.56) (xy 264.16 162.56)
 		)
 		(stroke
@@
 	(wire
 		(pts
-			(xy 281.94 116.84) (xy 298.45 116.84)
+			(xy 129.54 36.83) (xy 162.56 36.83)
 		)
 		(stroke
@@
 	(wire
 		(pts
-			(xy 203.2 83.82) (xy 203.2 147.32)
+			(xy 281.94 116.84) (xy 298.45 116.84)
 		)
 		(stroke
@@
 	(wire
 		(pts
-			(xy 237.49 62.23) (xy 189.23 62.23)
+			(xy 203.2 83.82) (xy 203.2 147.32)
 		)
 		(stroke
@@
 	(wire
 		(pts
-			(xy 205.74 168.91) (xy 158.75 168.91)
+			(xy 237.49 62.23) (xy 189.23 62.23)
 		)
 		(stroke
@@
 	(wire
 		(pts
-			(xy 83.82 161.29) (xy 83.82 181.61)
+			(xy 83.82 140.97) (xy 83.82 161.29)
 		)
 		(stroke
@@
 	(wire
 		(pts
-			(xy 226.06 168.91) (xy 226.06 170.18)
+			(xy 205.74 168.91) (xy 205.74 171.45)
 		)
 		(stroke
@@
 	(wire
 		(pts
+			(xy 226.06 137.16) (xy 226.06 154.94)
+		)
+		(stroke
+			(width 0)
+			(type default)
+		)
+	)
+	(wire
+		(pts
+			(xy 90.17 161.29) (xy 90.17 167.64)
+		)
+		(stroke
+			(width 0)
+			(type default)
+		)
+	)
+	(wire
+		(pts
 			(xy 218.44 118.11) (xy 218.44 92.71)
 		)
@@
 	(wire
 		(pts
-			(xy 95.25 161.29) (xy 96.52 161.29)
+			(xy 83.82 161.29) (xy 90.17 161.29)
 		)
 		(stroke
@@
 	(wire
 		(pts
+			(xy 205.74 168.91) (xy 208.28 168.91)
+		)
+		(stroke
+			(width 0)
+			(type default)
+		)
+	)
+	(wire
+		(pts
 			(xy 264.16 138.43) (xy 285.75 138.43)
 		)
@@
 	(wire
 		(pts
-			(xy 264.16 148.59) (xy 264.16 162.56)
+			(xy 90.17 161.29) (xy 104.14 161.29)
 		)
 		(stroke
@@
 	(wire
 		(pts
-			(xy 208.28 168.91) (xy 205.74 168.91)
+			(xy 264.16 148.59) (xy 264.16 162.56)
 		)
 		(stroke
@@
 	(wire
 		(pts
+			(xy 83.82 161.29) (xy 83.82 181.61)
+		)
+		(stroke
+			(width 0)
+			(type default)
+		)
+	)
+	(wire
+		(pts
 			(xy 248.92 185.42) (xy 266.7 185.42)
 		)
@@
 	(wire
 		(pts
-			(xy 83.82 181.61) (xy 104.14 181.61)
+			(xy 83.82 181.61) (xy 90.17 181.61)
 		)
 		(stroke
@@
 	(wire
 		(pts
-			(xy 104.14 163.83) (xy 104.14 161.29)
+			(xy 104.14 161.29) (xy 104.14 163.83)
 		)
 		(stroke
@@
 	(wire
 		(pts
+			(xy 96.52 58.42) (xy 96.52 181.61)
+		)
+		(stroke
+			(width 0)
+			(type default)
+		)
+	)
+	(wire
+		(pts
 			(xy 246.38 180.34) (xy 246.38 57.15)
 		)
@@
 	(wire
 		(pts
-			(xy 158.75 137.16) (xy 125.73 137.16)
+			(xy 125.73 137.16) (xy 226.06 137.16)
 		)
 		(stroke
@@
 	(wire
 		(pts
-			(xy 96.52 58.42) (xy 96.52 161.29)
-		)
-		(stroke
-			(width 0)
-			(type default)
-		)
-	)
-	(wire
-		(pts
 			(xy 137.16 160.02) (xy 130.81 160.02)
 		)
@@
 	(wire
 		(pts
-			(xy 83.82 140.97) (xy 83.82 161.29)
-		)
-		(stroke
-			(width 0)
-			(type default)
-		)
-	)
-	(wire
-		(pts
 			(xy 318.77 46.99) (xy 205.74 46.99)
 		)
@@
 	(wire
 		(pts
+			(xy 96.52 181.61) (xy 104.14 181.61)
+		)
+		(stroke
+			(width 0)
+			(type default)
+		)
+	)
+	(wire
+		(pts
 			(xy 63.5 102.87) (xy 68.58 102.87)
 		)
@@
 	(wire
 		(pts
-			(xy 83.82 161.29) (xy 87.63 161.29)
-		)
-		(stroke
-			(width 0)
-			(type default)
-		)
-	)
-	(wire
-		(pts
 			(xy 38.1 119.38) (xy 38.1 123.19)
 		)
@@
 	(wire
 		(pts
-			(xy 96.52 161.29) (xy 104.14 161.29)
-		)
-		(stroke
-			(width 0)
-			(type default)
-		)
-	)
-	(wire
-		(pts
 			(xy 66.04 72.39) (xy 66.04 80.01)
 		)
@@
 	(wire
 		(pts
-			(xy 158.75 168.91) (xy 158.75 137.16)
-		)
-		(stroke
-			(width 0)
-			(type default)
-		)
-	)
-	(wire
-		(pts
 			(xy 285.75 92.71) (xy 285.75 106.68)
 		)
@@
 	(wire
 		(pts
+			(xy 90.17 181.61) (xy 96.52 181.61)
+		)
+		(stroke
+			(width 0)
+			(type default)
+		)
+	)
+	(wire
+		(pts
 			(xy 41.91 90.17) (xy 41.91 88.9)
 		)
@@
 	(symbol
 		(lib_id "Diode:1N4007")
-		(at 91.44 161.29 0)
+		(at 90.17 171.45 90)
 		(unit 1)
 		(exclude_from_sim no)
@@
 		(fields_autoplaced yes)
 		(property "Reference" "D3"
-			(at 91.44 154.94 0)
+			(at 92.71 170.1799 90)
 			(effects
 				(font
 					(size 1.27 1.27)
 				)
+				(justify right)
 			)
 		)
 		(property "Value" "1N4007"
-			(at 91.44 157.48 0)
+			(at 92.71 172.7199 90)
 			(effects
 				(font
 					(size 1.27 1.27)
 				)
+				(justify right)
 			)
 		)
 		(property "Footprint" "Diode_THT:D_DO-41_SOD81_P10.16mm_Horizontal"
-			(at 91.44 165.735 0)
+			(at 94.615 171.45 0)
 			(effects
 				(font
@@
 		)
 		(property "Datasheet" "http://www.vishay.com/docs/88503/1n4001.pdf"
-			(at 91.44 161.29 0)
+			(at 90.17 171.45 0)
 			(effects
 				(font
@@
 		)
 		(property "Description" "1000V 1A General Purpose Rectifier Diode, DO-41"
-			(at 91.44 161.29 0)
+			(at 90.17 171.45 0)
 			(effects
 				(font
@@
 		)
 		(property "Sim.Device" "D"
-			(at 91.44 161.29 0)
+			(at 90.17 171.45 0)
 			(effects
 				(font
@@
 		)
 		(property "Sim.Pins" "1=K 2=A"
-			(at 91.44 161.29 0)
+			(at 90.17 171.45 0)
 			(effects
 				(font
@@
 		(lib_id "Diode:1N4007")
 		(at 274.32 92.71 0)
+		(mirror y)
 		(unit 1)
 		(exclude_from_sim no)
@@
 		(on_board yes)
 		(dnp no)
-		(fields_autoplaced yes)
 		(property "Reference" "D8"
 			(at 274.32 86.36 0)
@@
 		(lib_id "Diode:1N4007")
 		(at 274.32 148.59 0)
+		(mirror y)
 		(unit 1)
 		(exclude_from_sim no)
@@
 		(on_board yes)
 		(dnp no)
-		(fields_autoplaced yes)
 		(property "Reference" "D9"
 			(at 274.32 142.24 0)
@@
 		(lib_id "Diode:1N4007")
 		(at 215.9 154.94 0)
+		(mirror y)
 		(unit 1)
 		(exclude_from_sim no)
@@
 		(on_board yes)
 		(dnp no)
-		(fields_autoplaced yes)
 		(property "Reference" "D12"
 			(at 215.9 148.59 0)
@@
 	(symbol
 		(lib_id "power:GND")
-		(at 226.06 170.18 0)
+		(at 205.74 171.45 0)
 		(unit 1)
 		(exclude_from_sim no)
@@
 		(fields_autoplaced yes)
 		(property "Reference" "#PWR09"
-			(at 226.06 176.53 0)
+			(at 205.74 177.8 0)
 			(effects
 				(font
@@
 		)
 		(property "Value" "GND"
-			(at 226.06 175.26 0)
+			(at 205.74 176.53 0)
 			(effects
 				(font
@@
 		)
 		(property "Footprint" ""
-			(at 226.06 170.18 0)
+			(at 205.74 171.45 0)
 			(effects
 				(font
@@
 		)
 		(property "Datasheet" ""
-			(at 226.06 170.18 0)
+			(at 205.74 171.45 0)
 			(effects
 				(font
@@
 		)
 		(property "Description" "Power symbol creates a global label with name \"GND\" , ground"
-			(at 226.06 170.18 0)
+			(at 205.74 171.45 0)
 			(effects
 				(font
