File: arduino/kicad/unoQ/greenlight-tester-unoQ.kicad_sch (KiCad schematic)
At the start: 42 parts, among them J1 AudioJack2, J1 Conn_01x08, J2 AudioJack2, J2 Conn_01x10, J3 Conn_01x06, J3 XLR3, J4 Conn_01x08, J4 XLR3, K1 Relay_DPDT, K2 Relay_DPDT, K3 Relay_DPDT, K4 Relay_DPDT, K5 Relay_DPDT, K6 Relay_DPDT, Q1 PN2222A, Q2 PN2222A, Q3 PN2222A, Q4 PN2222A, Q5 PN2222A, Q6 PN2222A

Commit message: first pass at UPC handling
Parts:
- removed J4: Conn_01x08, symbol Connector_Generic:Conn_01x08
- added D7: LED, symbol Device:LED
- added J6: Conn_01x08, symbol Connector_Generic:Conn_01x08
- added R13: R220, Resistor_THT:R_Axial_DIN0204_L3.6mm_D1.6mm_P1.90mm_Vertical, symbol Device:R
- renumbered D6 to D1, D5 to D2, D12 to D4, D8 to D5, D9 to D6, Q5 to Q4, Q6 to Q5, Q4 to Q6, R11 to R10, R12 to R11, R2 to R12, R10 to R2, R9 to R3, R3 to R4, R4 to R5, R13 to R6, R15 to R7, R14 to R8, R8 to R9
Connections:
- net A1 is gone; now on net A1/D15: J3.5 (A1)
- net +3V3: now also J6.5 (3.3V)
- net 5V: now also D1.1 (K), D2.1 (K), D3.1 (K), D4.1 (K), J6.4 (5V); no longer D1.2 (A), D2.2 (A), D3.2 (A), D4.2 (A)
- net D10: now also R8.1; no longer R10.1
- net D11: now also R9.1; no longer R11.1
- net D12: now also R7.1; no longer J3.1
- net D13: now also R1.1; no longer K5.22
- net D2: now also D7.2 (A); no longer K1.14
- net D4: now also R11.2; no longer K2.14, R2.2
- net D5: now also R10.1; no longer K2.24, R3.2
- net D6: now also K1.14; no longer R1.1
- net D7: now also K1.24; no longer R7.1
- net D8: now also K2.14, R2.2; no longer R8.1
- net D9: now also K2.24, R3.2; no longer R9.1
- net GND: now also J6.2 (GND), J6.3 (GND), R13.1
- net RST: now also J6.6 (RST)
- net VIN: now also J6.1 (Vin)
- net at K3.A2, Q3.3 (C): now also D3.2 (A); no longer D3.1 (K)
- net at K1.A2, K2.A2, Q2.3 (C): now also D1.2 (A), D2.2 (A); no longer D1.1 (K), D2.1 (K)
- net at K4.11: now also K3.14; no longer K3.24
- net at K4.21: now also K3.24; no longer K3.14
- net at K4.A2, Q4.3 (C): now also D4.2 (A); no longer D4.1 (K)
- net at Q6.2 (B): now also R11.1; no longer R11.2
- net A1/D15: now reaches K6.22
- net A2 renamed A2/D16
- net A2/D16: now also K5.22
- net A3 renamed A3/D17
- net A3/D17: now also K6.12; no longer J4.1
- net A4 renamed A4/D18
- net A5 renamed A5/D19
- net A5/D19: now also J1.4 (D3), J3.1, J4.1; no longer K6.12
- net AREF: no longer names the net of J2.8 (AREF)
- net D0: no longer names the net of J1.1 (D0)
- net D1: no longer names the net of J1.2 (D1)
- removed net D3: J1.4 (D3), K1.24
- net SCL1 renamed D21
- net SDA1 renamed D20
- new net: D7.1 (K), R13.2
- no-connect marks 2 -> 5
Other:
- moved on the sheet: D4, D6, K4, K6, Q1, Q2, Q4, Q5, Q6, R1, R10, R11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
